Commit message: Fixed handles frames

File: src/project_name_/urdf/handle.xacro (robot description, xacro)
@@ -48,4 +48,5 @@
         <!-- handle -->
         <joint name="${parent}_${name}_handle_joint" type="fixed">
+            <origin xyz="-${bar_length} 0 0" rpy="1.57 0 0"/>
             <parent link="${name}_base_link"/>
             <child link="${name}_handle"/>
@@ -53,5 +54,5 @@
         <link name="${name}_handle">
             <visual>
-                <origin xyz="-${bar_length} 0 0" rpy="1.57 0 0" />
+                <!-- <origin xyz="-${bar_length} 0 0" rpy="1.57 0 0" /> -->
                 <geometry>
                     <cylinder radius="${handle_radius}" length="${handle_length}" />

Commit message: Changed handles orientation

File: src/project_name_/urdf/handle.xacro (robot description, xacro)
@@ -21,5 +21,5 @@
         <link name="${name}_leftBar">
             <visual>
-                <origin xyz="-${bar_length/2} -${0.3*handle_length} 0" rpy="0 1.57 0" />
+                <origin xyz="-${bar_length/2} -${0*handle_length} 0" rpy="0 1.57 0" />
                 <geometry>
                     <cylinder radius="${bar_radius}" length="${bar_length}" />
@@ -37,5 +37,5 @@
         <link name="${name}_rightBar">
             <visual>
-                <origin xyz="-${bar_length/2} ${0.3*handle_length} 0" rpy="0 1.57 0" />
+                <origin xyz="-${bar_length/2} ${0*handle_length} 0" rpy="0 1.57 0" />
                 <geometry>
                     <cylinder radius="${bar_radius}" length="${bar_length}" />
@@ -54,5 +54,5 @@
         <link name="${name}_handle">
             <visual>
-                <!-- <origin xyz="-${bar_length} 0 0" rpy="1.57 0 0" /> -->
+                <origin xyz="0 ${0.5*bar_length} 0" rpy="1.57 0 0" />
                 <geometry>
                     <cylinder radius="${handle_radius}" length="${handle_length}" />
